File: PCB/html_accelerator/eMMC1.kicad_sch (KiCad schematic)
At the start: 8 parts, among them U10 MX30LF1G28AD-TI, U2 AU6438BS, U3 MX30LF1G28AD-TI, U4 AU6438BS, U5 AU6438BS, U7 AU6438BS, U8 MX30LF1G28AD-TI, U9 MX30LF1G28AD-TI

Commit message: EMMC symbol and footprint update
Parts:
- removed U10, U3, U8, U9: MX30LF1G28AD-TI, html_accel_footprints:MX30LF1G28AD-TI, symbol html_accel_Symbols:MX30LF1G28AD-TI
- removed U4, U5, U7: AU6438BS, Package_SO:SSOP-28_3.9x9.9mm_P0.635mm, symbol html_accel_Symbols:AU6438BS
- added U3, U4, U5: EMMC_4G, EMMC04G-M627-X03U_KNT, symbol html_accel_Symbols:EMMC_4G
