File: PCB/html_accelerator/PCIE_POWER.kicad_sch (KiCad schematic)
At the start: 28 parts, among them U1 MCS9990

Commit message: gerbers and readme updates
Parts:
- C5: symbol Device:C_Polarized_US -> Device:C
Other:
- company: (none) -> Spencer K
- title: 12v, 3v3, 1v2 Power, Buck -> HTML Accelerator
Changed lines of the file:
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@@
 	(paper "A4")
 	(title_block
-		(title "12v, 3v3, 1v2 Power, Buck")
-		(date "2024-09-15")
-		(rev "1")
+		(title "HTML Accelerator")
+		(date "2026-04-25")
+		(rev "1.0")
+		(company "Spencer K")
+		(comment 1 "https://github.com/akaStanley/HTML_Accelerator")
 	)
 	(junction
@@
 	)
 	(symbol
-		(lib_id "Device:C_Polarized_US")
+		(lib_id "Device:C")
 		(at 184.15 58.42 0)
 		(mirror y)
@@
 		)
 		(property "Footprint" "Capacitor_SMD:C_0805_2012Metric_Pad1.18x1.45mm_HandSolder"
-			(at 184.15 58.42 0)
+			(at 183.1848 62.23 0)
 			(hide yes)
 			(show_name no)
@@
 			)
 		)
-		(property "Description" ""
+		(property "Description" "Unpolarized capacitor"
 			(at 184.15 58.42 0)
-			(show_name no)
-			(do_not_autoplace no)
+			(hide yes)
+			(show_name no)
+			(do_not_autoplace no)
