File: PCB/html_accelerator/eMMC2.kicad_sch (KiCad schematic)
At the start: 15 parts, among them U5 EMMC_4G, U6 EMMC_4G, U8 AU6438BS, Y3 12MHz

Commit message: gerbers and readme updates
Parts:
- U5, U6: value EMMC_4G -> H26M31003
Other:
- company: (none) -> Spencer K
- title: (none) -> HTML Accelerator
Changed lines of the file:
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@@
 	(generator_version "10.0")
 	(paper "A4")
+	(title_block
+		(title "HTML Accelerator")
+		(date "2026-04-25")
+		(rev "1.0")
+		(company "Spencer K")
+		(comment 1 "https://github.com/akaStanley/HTML_Accelerator")
+	)
 	(text "4.7uF for VCC/VSS"
 		(exclude_from_sim no)
@@
 			)
 		)
-		(property "Value" "EMMC_4G"
+		(property "Value" "H26M31003"
 			(at 224.79 47.2581 0)
 			(show_name no)
@@
 			)
 		)
-		(property "Value" "EMMC_4G"
+		(property "Value" "H26M31003"
 			(at 172.72 47.2581 0)
 			(show_name no)
@@
 			)
 		)
-		(property "Value" "EMMC_4G"
+		(property "Value" "H26M31003"
 			(at 262.89 47.2581 0)
 			(show_name no)

Commit message: updated gerbers for fab
Parts:
- C47, C48: value 22pF -> 20pF
Changed lines of the file:
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@@
 	(title_block
 		(title "HTML Accelerator")
-		(date "2026-04-25")
+		(date "2026-04-29")
 		(rev "1.0")
 		(company "Spencer K")
@@
 			)
 		)
-		(property "Value" "22pF"
+		(property "Value" "20pF"
 			(at 44.45 104.14 0)
 			(show_name no)
@@
 			)
 		)
-		(property "Value" "22pF"
+		(property "Value" "20pF"
 			(at 29.21 104.14 0)
 			(show_name no)
